File: Hardware/Panel/mikrokosmos-ii-panel/mikrokosmos-ii-panel.kicad_sch (KiCad schematic)
At the start: 9 parts

Commit message: panel, PCB updates
Parts:
- added GRAF5: Art inverted, mikrokosmos-ii-panel:mikrokosmos-ii_panel_inv_art, symbol ao_symbols:Graphic
- added H6: Mounting_Hole, Kosmo_panel:Kosmo_Panel_Mounting_Hole, symbol Kosmo:Mounting_Hole
- GRAF1: footprint mikrokosmos-ii-panel:mikrokosmos-ii-panel-holes -> mikrokosmos-ii-panel:mikrokosmos-ii_panel_holes
- GRAF2: footprint mikrokosmos-ii-panel:mikrokosmos-ii-panel-art -> mikrokosmos-ii-panel:mikrokosmos-ii_panel_art
- GRAF3: value CC0 logo -> Art for Cu; footprint ao_tht:CC0_logo -> mikrokosmos-ii-panel:mikrokosmos-ii_panel_artc
- GRAF4: footprint mikrokosmos-ii-panel:mikrokosmos-ii-panel-artc -> mikrokosmos-ii-panel:mikrokosmos-ii_panel_artc
Connections:
- net GND: no longer H3.1
- no-connect marks 0 -> 2
Changed lines of the file:
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@@
     (comment 2 "To the extent possible under law, Richard Holmes has waived all copyright and related ")
   )
+  (no_connect (at 114.3 54.61))
+  (no_connect (at 88.9 54.61))
   (image (at 254 184.15) (scale 0.3)
     (data
@@
       (effects (font (size 1.27 1.27)) (justify left))
     )
-    (property "Footprint" "mikrokosmos-ii-panel:mikrokosmos-ii-panel-holes" (id 2) (at 175.26 50.8 0)
+    (property "Footprint" "mikrokosmos-ii-panel:mikrokosmos-ii_panel_holes" (id 2) (at 175.26 50.8 0)
       (effects (font (size 1.27 1.27)) hide)
     )
@@
       (effects (font (size 1.27 1.27)) (justify left))
     )
-    (property "Footprint" "mikrokosmos-ii-panel:mikrokosmos-ii-panel-art" (id 2) (at 175.26 57.15 0)
+    (property "Footprint" "mikrokosmos-ii-panel:mikrokosmos-ii_panel_art" (id 2) (at 175.26 57.15 0)
       (effects (font (size 1.27 1.27)) hide)
     )
@@
     )
   )
-  (symbol (lib_id "ao_symbols:Graphic") (at 175.26 63.5 0) (unit 1)
-    (in_bom yes) (on_board yes)
-    (property "Reference" "GRAF3" (id 0) (at 182.3212 62.3316 0)
-      (effects (font (size 1.27 1.27)) (justify left))
-    )
-    (property "Value" "CC0 logo" (id 1) (at 182.3212 64.643 0)
-      (effects (font (size 1.27 1.27)) (justify left))
-    )
-    (property "Footprint" "ao_tht:CC0_logo" (id 2) (at 175.26 63.5 0)
-      (effects (font (size 1.27 1.27)) hide)
-    )
-    (property "Datasheet" "" (id 3) (at 175.26 63.5 0)
-      (effects (font (size 1.27 1.27)) hide)
-    )
-    (property "Config" "DNF" (id 4) (at 175.26 63.5 0)
-      (effects (font (size 1.27 1.27)) hide)
-    )
+  (symbol (lib_id "Kosmo:Mounting_Hole") (at 114.3 52.07 0) (unit 1)
+    (in_bom yes) (on_board yes) (fields_autoplaced)
+    (property "Reference" "H6" (id 0) (at 116.84 49.9653 0)
+      (effects (font (size 1.27 1.27)) (justify left))
+    )
+    (property "Value" "Mounting_Hole" (id 1) (at 116.84 52.5022 0)
+      (effects (font (size 1.27 1.27)) (justify left))
+    )
+    (property "Footprint" "Kosmo_panel:Kosmo_Panel_Mounting_Hole" (id 2) (at 114.3 52.07 0)
+      (effects (font (size 1.27 1.27)) hide)
+    )
+    (property "Datasheet" "" (id 3) (at 114.3 52.07 0)
+      (effects (font (size 1.27 1.27)) hide)
+    )
+    (pin "1")
   )
   (symbol (lib_id "ao_symbols:Graphic") (at 196.85 57.15 0) (unit 1)
@@
       (effects (font (size 1.27 1.27)) (justify left))
     )
-    (property "Footprint" "mikrokosmos-ii-panel:mikrokosmos-ii-panel-artc" (id 2) (at 196.85 57.15 0)
+    (property "Footprint" "mikrokosmos-ii-panel:mikrokosmos-ii_panel_artc" (id 2) (at 196.85 57.15 0)
       (effects (font (size 1.27 1.27)) hide)
     )
@@
     (pin "1")
   )
-  (symbol (lib_id "power:GND") (at 88.9 54.61 0) (unit 1)
-    (in_bom yes) (on_board yes) (fields_autoplaced)
-    (property "Reference" "#PWR03" (id 0) (at 88.9 60.96 0)
-      (effects (font (size 1.27 1.27)) hide)
-    )
-    (property "Value" "GND" (id 1) (at 88.9 59.0534 0))
-    (property "Footprint" "" (id 2) (at 88.9 54.61 0)
-      (effects (font (size 1.27 1.27)) hide)
-    )
-    (property "Datasheet" "" (id 3) (at 88.9 54.61 0)
-      (effects (font (size 1.27 1.27)) hide)
-    )
-    (pin "1")
+  (symbol (lib_id "ao_symbols:Graphic") (at 196.85 63.5 0) (unit 1)
+    (in_bom yes) (on_board yes)
+    (property "Reference" "GRAF3" (id 0) (at 203.9112 62.3316 0)
+      (effects (font (size 1.27 1.27)) (justify left))
+    )
+    (property "Value" "Art for Cu" (id 1) (at 203.9112 64.643 0)
+      (effects (font (size 1.27 1.27)) (justify left))
+    )
+    (property "Footprint" "mikrokosmos-ii-panel:mikrokosmos-ii_panel_artc" (id 2) (at 196.85 63.5 0)
+      (effects (font (size 1.27 1.27)) hide)
+    )
+    (property "Datasheet" "" (id 3) (at 196.85 63.5 0)
+      (effects (font (size 1.27 1.27)) hide)
+    )
+    (property "Config" "DNF" (id 4) (at 196.85 63.5 0)
+      (effects (font (size 1.27 1.27)) hide)
+    )
+  )
+  (symbol (lib_id "ao_symbols:Graphic") (at 196.85 50.8 0) (unit 1)
+    (in_bom yes) (on_board yes)
+    (property "Reference" "GRAF5" (id 0) (at 203.9112 49.6316 0)
+      (effects (font (size 1.27 1.27)) (justify left))
+    )
+    (property "Value" "Art inverted" (id 1) (at 203.9112 51.943 0)
+      (effects (font (size 1.27 1.27)) (justify left))
+    )
+    (property "Footprint" "mikrokosmos-ii-panel:mikrokosmos-ii_panel_inv_art" (id 2) (at 196.85 50.8 0)
+      (effects (font (size 1.27 1.27)) hide)
+    )
+    (property "Datasheet" "" (id 3) (at 196.85 50.8 0)
+      (effects (font (size 1.27 1.27)) hide)
+    )
+    (property "Config" "DNF" (id 4) (at 196.85 50.8 0)
+      (effects (font (size 1.27 1.27)) hide)
+    )
   )
   (sheet_instances
@@
       (reference "#PWR02") (unit 1) (value "GND") (footprint "")
     )
-    (path "/6bbb3837-2584-429d-8342-6d7a0c841443"
-      (reference "#PWR03") (unit 1) (value "GND") (footprint "")
-    )
     (path "/00000000-0000-0000-0000-00005f0c12be"
       (reference "#PWR04") (unit 1) (value "GND") (footprint "")
@@
     )
     (path "/00000000-0000-0000-0000-000061599166"
-      (reference "GRAF1") (unit 1) (value "Holes") (footprint "mikrokosmos-ii-panel:mikrokosmos-ii-panel-holes")
+      (reference "GRAF1") (unit 1) (value "Holes") (footprint "mikrokosmos-ii-panel:mikrokosmos-ii_panel_holes")
     )
     (path "/00000000-0000-0000-0000-0000615997cb"
-      (reference "GRAF2") (unit 1) (value "Art") (footprint "mikrokosmos-ii-panel:mikrokosmos-ii-panel-art")
-    )
-    (path "/00000000-0000-0000-0000-00006159994e"
-      (reference "GRAF3") (unit 1) (value "CC0 logo") (footprint "ao_tht:CC0_logo")
+      (reference "GRAF2") (unit 1) (value "Art") (footprint "mikrokosmos-ii-panel:mikrokosmos-ii_panel_art")
+    )
+    (path "/b5e0b9e9-8f17-4422-bf34-cabcbc7bf23a"
+      (reference "GRAF3") (unit 1) (value "Art for Cu") (footprint "mikrokosmos-ii-panel:mikrokosmos-ii_panel_artc")
     )
     (path "/4924a5c9-3a6d-4b5c-a4e1-688957905b45"
-      (reference "GRAF4") (unit 1) (value "Art for Cu") (footprint "mikrokosmos-ii-panel:mikrokosmos-ii-panel-artc")
+      (reference "GRAF4") (unit 1) (value "Art for Cu") (footprint "mikrokosmos-ii-panel:mikrokosmos-ii_panel_artc")
+    )
+    (path "/baf9e44b-c22d-493e-9c00-45957b38efff"
+      (reference "GRAF5") (unit 1) (value "Art inverted") (footprint "mikrokosmos-ii-panel:mikrokosmos-ii_panel_inv_art")
     )
     (path "/00000000-0000-0000-0000-00005f0bcd70"
@@
       (reference "H5") (unit 1) (value "Mounting_Holes") (footprint "Kosmo_panel:Kosmo_Panel_Dual_Slotted_Mounting_Holes")
     )
-  )
+    (path "/3f3726d1-900a-4746-95fa-2c28bdb226ed"
+      (reference "H6") (unit 1) (value "Mounting_Hole") (footprint "Kosmo_panel:Kosmo_Panel_Mounting_Hole")
+    )
+  )
