File: Hardware/PCB/mikrokosmos-ii/mikrokosmos-ii.kicad_pcb (KiCad board)
At the start: 2 copper layers, 21 x 121 mm, 28 parts, among them J2 Synth_power_2x5, J3 2_pin_Molex_header, J7 2_pin_Molex_header, U1 TL072

Commit message: README, reorient capacitor
Parts:
- moved C2 1.80 mm to (106.3, 32.7), turned to 90 degrees
Routing:
- net +12V: track 57.5 -> 58.6 mm
Changed lines of the file:
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@@
   )
   (footprint "ao_tht:CP_Radial_D6.3mm_P2.50mm" (layer "B.Cu")
-    (at 107.62 31.42 180)
+    (at 106.35 32.69 90)
     (descr "CP, Radial series, Radial, pin pitch=2.50mm, , diameter=6.3mm, Electrolytic Capacitor")
     (tags "CP Radial series Radial pin pitch 2.50mm  diameter 6.3mm Electrolytic Capacitor")
@@
     (property "Vendor" "Tayda")
     (attr through_hole)
-    (fp_text reference "C2" (at -1 4.4 180) (layer "B.SilkS")
-      (effects (font (size 0.75 0.75) (thickness 0.15)) (justify mirror))
-    )
-    (fp_text value "10uF" (at 1.25 -4.4 180) (layer "B.Fab")
-      (effects (font (size 1 1) (thickness 0.15)) (justify mirror))
-    )
-    (fp_text user "${VALUE}" (at 4 4.5 180) (layer "B.SilkS")
-      (effects (font (size 0.75 0.75) (thickness 0.15)) (justify mirror))
-    )
-    (fp_text user "${REFERENCE}" (at 1.25 0 180) (layer "B.Fab")
+    (fp_text reference "C2" (at -1 4.4 90) (layer "B.SilkS")
+      (effects (font (size 0.75 0.75) (thickness 0.15)) (justify mirror))
+    )
+    (fp_text value "10uF" (at 1.25 -4.4 90) (layer "B.Fab")
+      (effects (font (size 1 1) (thickness 0.15)) (justify mirror))
+    )
+    (fp_text user "${VALUE}" (at 4 4.5 90) (layer "B.SilkS")
+      (effects (font (size 0.75 0.75) (thickness 0.15)) (justify mirror))
+    )
+    (fp_text user "${REFERENCE}" (at 1.25 0 90) (layer "B.Fab")
       (effects (font (size 1 1) (thickness 0.15)) (justify mirror))
     )
@@
     (fp_line (start -1.443972 1.3735) (end -0.813972 1.3735) (layer "B.Fab") (width 0.1))
     (fp_circle (center 1.25 0) (end 4.4 0) (layer "B.Fab") (width 0.1) (fill none))
-    (pad "1" thru_hole rect locked (at 0 0 180) (size 1.6 1.6) (drill 0.8) (layers *.Cu *.Mask)
+    (pad "1" thru_hole rect locked (at 0 0 90) (size 1.6 1.6) (drill 0.8) (layers *.Cu *.Mask)
       (net 1 "+12V") (pintype "passive"))
-    (pad "2" thru_hole circle locked (at 2.5 0 180) (size 1.6 1.6) (drill 0.8) (layers *.Cu *.Mask)
+    (pad "2" thru_hole circle locked (at 2.5 0 90) (size 1.6 1.6) (drill 0.8) (layers *.Cu *.Mask)
       (net 2 "GND") (pintype "passive"))
     (model "${KICAD_AOKICAD}/ao_tht_3d/CP_Radial_D6.3mm_P2.50mm.wrl"
@@
     (style (thickness 0.1) (arrow_length 1.27) (text_position_mode 0) (extension_height 0.58642) (extension_offset 0.5) keep_text_aligned)
   )
-  (segment (start 108.994511 71.965489) (end 108.994511 32.794511) (width 0.75) (layer "F.Cu") (net 1))
-  (segment (start 108.06 30.98) (end 107.62 31.42) (width 0.75) (layer "F.Cu") (net 1))
-  (segment (start 108.06 26.34) (end 108.06 30.98) (width 0.75) (layer "F.Cu") (net 1))
-  (segment (start 103.81 77.15) (end 103.82 77.14) (width 0.75) (layer "F.Cu") (net 1))
+  (segment (start 103.82 77.14) (end 108.994511 71.965489) (width 0.75) (layer "F.Cu") (net 1))
+  (segment (start 108.994511 35.334511) (end 106.35 32.69) (width 0.75) (layer "F.Cu") (net 1))
+  (segment (start 108.06 30.98) (end 108.06 26.34) (width 0.75) (layer "F.Cu") (net 1))
   (segment (start 103.81 80.96) (end 103.81 77.15) (width 0.75) (layer "F.Cu") (net 1))
-  (segment (start 108.994511 32.794511) (end 107.62 31.42) (width 0.75) (layer "F.Cu") (net 1))
-  (segment (start 103.82 77.14) (end 108.994511 71.965489) (width 0.75) (layer "F.Cu") (net 1))
+  (segment (start 106.35 32.69) (end 108.06 30.98) (width 0.75) (layer "F.Cu") (net 1))
+  (segment (start 108.994511 71.965489) (end 108.994511 35.334511) (width 0.75) (layer "F.Cu") (net 1))
   (segment (start 103.79 35.25) (end 94.412 44.628) (width 0.75) (layer "F.Cu") (net 3))
   (segment (start 94.412 63.902) (end 96.23 65.72) (width 0.75) (layer "F.Cu") (net 3))
@@
   (segment (start 102.135489 17.854511) (end 102.135489 33.595489) (width 0.75) (layer "F.Cu") (net 3))
   (segment (start 94.412 44.628) (end 94.412 63.902) (width 0.75) (layer "F.Cu") (net 3))
-  (segment (start 96.23 69.49) (end 96.2 69.52) (width 0.75) (layer "F.Cu") (net 3))
   (segment (start 91.255489 76.025489) (end 92.38 77.15) (width 0.25) (layer "F.Cu") (net 4))
   (segment (start 91.255489 63.034511) (end 91.255489 76.025489) (width 0.25) (layer "F.Cu") (net 4))
   (segment (start 92.38 61.91) (end 91.255489 63.034511) (width 0.25) (layer "F.Cu") (net 4))
   (segment (start 92.38 77.15) (end 92.38 80.92) (width 0.25) (layer "F.Cu") (net 4))
-  (segment (start 92.38 80.92) (end 92.42 80.96) (width 0.25) (layer "F.Cu") (net 4))
-  (segment (start 96.19 77.15) (end 96.2 77.14) (width 0.25) (layer "B.Cu") (net 4))
   (segment (start 92.38 77.15) (end 96.19 77.15) (width 0.25) (layer "B.Cu") (net 4))
   (segment (start 97.724511 76.124511) (end 97.724511 80.655489) (width 0.25) (layer "F.Cu") (net 5))
@@
   (segment (start 92.38 66.99) (end 92.38 70.78) (width 0.25) (layer "F.Cu") (net 5))
   (segment (start 92.38 70.78) (end 96.2 74.6) (width 0.25) (layer "F.Cu") (net 5))
-  (segment (start 97.724511 80.655489) (end 97.42 80.96) (width 0.25) (layer "F.Cu") (net 5))
   (segment (start 98.73 122.86) (end 105.08 129.21) (width 0.25) (layer "F.Cu") (net 5))
   (segment (start 96.2 74.6) (end 97.724511 76.124511) (width 0.25) (layer "F.Cu") (net 5))
@@
   (segment (start 98.584511 49.054511) (end 104.934511 49.054511) (width 0.25) (layer "B.Cu") (net 6))
   (segment (start 104.934511 49.054511) (end 107.62 51.74) (width 0.25) (layer "B.Cu") (net 6))
-  (segment (start 102.54 47.97) (end 102.58 47.93) (width 0.25) (layer "F.Cu") (net 7))
   (segment (start 102.54 51.74) (end 102.54 47.97) (width 0.25) (layer "F.Cu") (net 7))
   (segment (start 102.54 51.74) (end 102.54 56.82) (width 0.25) (layer "F.Cu") (net 7))
@@
   (segment (start 103.82 74.6) (end 107.62 78.4) (width 0.25) (layer "B.Cu") (net 8))
   (segment (start 107.62 78.4) (end 107.62 79.69) (width 0.25) (layer "B.Cu") (net 8))
-  (segment (start 107.62 65.76) (end 107.58 65.72) (width 0.25) (layer "F.Cu") (net 9))
   (segment (start 102.29548 80.35518) (end 102.54 80.5997) (width 0.25) (layer "F.Cu") (net 9))
   (segment (start 102.54 80.5997) (end 102.54 86.03) (width 0.25) (layer "F.Cu") (net 9))
@@
   (segment (start 102.54 61.9) (end 102.54 63.5003) (width 0.25) (layer "F.Cu") (net 13))
   (segment (start 92.38 51.75) (end 97.45 51.75) (width 0.25) (layer "B.Cu") (net 13))
-  (segment (start 97.45 51.75) (end 97.46 51.74) (width 0.25) (layer "B.Cu") (net 13))
   (segment (start 93.65 133.02) (end 97.46 129.21) (width 0.25) (layer "F.Cu") (net 14))
   (segment (start 92.38 133.02) (end 93.65 133.02) (width 0.25) (layer "F.Cu") (net 14))

Commit message: Small refinements to layout and schem
Parts:
- added TP1: +12V, ao_tht:TestPoint_THTPad_D1.5mm_Drill0.7mm, F.Cu at (91.1, 36.5)
- added TP2: GND, ao_tht:TestPoint_THTPad_1.5x1.5mm_Drill0.7mm, F.Cu at (91.1, 40.3)
- added TP3: -12V, ao_tht:TestPoint_THTPad_D1.5mm_Drill0.7mm, F.Cu at (91.1, 44.1)
- C5, C6: footprint Capacitor_THT:C_Disc_D3.0mm_W1.6mm_P2.50mm -> ao_tht:C_Disc_D3.0mm_W1.6mm_P2.50mm
Routing:
- net +12V: track 58.6 -> 75.4 mm
- net -12V: track 62.9 -> 66.5 mm
- net Net-(C11-Pad2): track 48.8 -> 49.3 mm
Other:
- board text added: "Piezo in"
- board text added: "Preamp out"

Commit message: PCB touchup, reorg files, panel
Parts:
- added GRAF2: CC0 logo, ao_tht:CC0_logo, B.Cu at (94.7, 102.9)
- added GRAF3: AO logo, ao_tht:analogoutput, B.Cu at (100.0, 112.3)
Other:
- board text added: "GND / IN"
- board text added: "GND / OUT"
- board text added: "MIKROKOSMOS II Rich Holmes 7/2022 CC0 1.0"
- board text added: "https://github.com/holmesrichards/mikrokosmosii"
- board text removed: "Piezo in"
- board text removed: "Preamp out"

Commit message: panel, PCB updates
Parts:
- added H2: MountingHole, ao_tht:MountingHole_3.2mm_M3, F.Cu at (100.0, 92.0)
- moved R6 6.35 mm to (92.4, 96.2), turned to 90 degrees
- moved R4 5.24 mm to (107.6, 84.8), turned to -90 degrees
- moved C11 5.11 mm to (102.5, 86.0), turned to 90 degrees
- moved GRAF2 5.00 mm to (94.7, 107.9)
- moved GRAF3 5.00 mm to (100.0, 117.3)
- moved J3 5.00 mm to (100.0, 134.2)
- moved J7 5.00 mm to (107.6, 134.2)
- moved R7 5.00 mm to (92.4, 138.0)
- moved R8 5.00 mm to (97.5, 127.9)
- moved RV1 5.00 mm to (100.0, 115.0)
Routing:
- net Net-(R4-Pad2): track 15.0 -> 9.31 mm
- net Net-(D3-Pad1): track 52.6 -> 57.6 mm
- net /PIEZO_IN: track 71.3 -> 76.3 mm
- net Net-(C10-Pad1): track 24.2 -> 25.8 mm
- net Net-(C10-Pad2): track 23.3 -> 24.8 mm
Other:
- board size 21 x 121 mm -> 21 x 126 mm

Commit message: Pre fab tweaks, Gerbers, cap descriptions
Parts:
- renumbered C2 to C1, C3 to C2, C1 to C3, C5 to C4, C6 to C5, C4 to C6, C10 to C8, C11 to C9, J7 to J4, J3 to J6, R8 to R1, R1 to R2, R2 to R3, R3 to R4, R4 to R5, R5 to R6, R6 to R7, R7 to R8
Routing:
- net Net-(C9-Pad2): track 48.9 -> 48.0 mm
Other:
- board text added: "from circuit by G.-W. Raes"
