File: Hardware/PCB/mikrokosmos-ii/mikrokosmos-ii.kicad_sch (KiCad schematic)
At the start: 33 parts, among them J1 AudioJack2_SwitchT, J2 Synth_power_2x5, J3 2_pin_Molex_header, J4 2_pin_Molex_connector, J5 AudioJack2, J6 2_pin_Molex_connector, J7 2_pin_Molex_header, U1 TL072

Commit message: Small refinements to layout and schem
Parts:
- added TP1: +12V, ao_tht:TestPoint_THTPad_D1.5mm_Drill0.7mm, symbol ao_symbols:TestPoint
- added TP2: GND, ao_tht:TestPoint_THTPad_1.5x1.5mm_Drill0.7mm, symbol ao_symbols:TestPoint
- added TP3: -12V, ao_tht:TestPoint_THTPad_D1.5mm_Drill0.7mm, symbol ao_symbols:TestPoint
- C5, C6: footprint Capacitor_THT:C_Disc_D3.0mm_W1.6mm_P2.50mm -> ao_tht:C_Disc_D3.0mm_W1.6mm_P2.50mm
Connections:
- net +12V: now also TP1.1
- net -12V: now also TP3.1
- net GND: now also TP2.1
Other:
- moved on the sheet: C2, C3, C5, C6, D1, D2, H1, J2, U1C

Commit message: Vendors
Parts:
- J2, R1, R2, R3, R4, R5, R7, U1: Vendor (none) -> Tayda
Changed lines of the file:
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@@
       (effects (font (size 1.524 1.524)) hide)
+    )
+    (property "Vendor" "Tayda" (id 4) (at 40.64 165.1 0)
+      (effects (font (size 1.27 1.27)) hide)
     )
     (pin "1")
@@
       (effects (font (size 1.27 1.27)) hide)
     )
+    (property "Vendor" "Tayda" (id 4) (at 105.41 80.01 0)
+      (effects (font (size 1.27 1.27)) hide)
+    )
     (pin "1")
     (pin "2")
@@
       (effects (font (size 1.27 1.27)) hide)
     )
+    (property "Vendor" "Tayda" (id 4) (at 105.41 91.44 0)
+      (effects (font (size 1.27 1.27)) hide)
+    )
     (pin "1")
     (pin "2")
@@
       (effects (font (size 1.27 1.27)) hide)
     )
+    (property "Vendor" "Tayda" (id 4) (at 123.19 80.01 0)
+      (effects (font (size 1.27 1.27)) hide)
+    )
     (pin "1")
     (pin "2")
@@
       (effects (font (size 1.27 1.27)) hide)
     )
+    (property "Vendor" "Tayda" (id 4) (at 137.16 92.71 0)
+      (effects (font (size 1.27 1.27)) hide)
+    )
     (pin "1")
     (pin "2")
@@
       (effects (font (size 1.27 1.27)) hide)
     )
+    (property "Vendor" "Tayda" (id 4) (at 168.275 85.09 0)
+      (effects (font (size 1.27 1.27)) hide)
+    )
     (pin "1")
     (pin "2")
@@
     )
     (property "Datasheet" "http://www.ti.com/lit/ds/symlink/tl071.pdf" (id 3) (at 186.055 82.55 0)
+      (effects (font (size 1.27 1.27)) hide)
+    )
+    (property "Vendor" "Tayda" (id 4) (at 186.055 82.55 0)
       (effects (font (size 1.27 1.27)) hide)
     )
@@
       (effects (font (size 1.27 1.27)) hide)
     )
+    (property "Vendor" "Tayda" (id 4) (at 186.055 93.98 0)
+      (effects (font (size 1.27 1.27)) hide)
+    )
     (pin "1")
     (pin "2")
@@
       (effects (font (size 1.27 1.27)) hide)
     )
+    (property "Vendor" "Tayda" (id 4) (at 215.265 82.55 0)
+      (effects (font (size 1.27 1.27)) hide)
+    )
     (pin "1")
     (pin "2")
@@
       (effects (font (size 1.27 1.27)) hide)
     )
+    (property "Vendor" "Tayda" (id 4) (at 128.27 165.1 0)
+      (effects (font (size 1.27 1.27)) hide)
+    )

Commit message: PCB touchup, reorg files, panel
Parts:
- added GRAF2: CC0 logo, ao_tht:CC0_logo, symbol ao_symbols:Graphic
- added GRAF3: AO logo, ao_tht:analogoutput, symbol ao_symbols:Graphic
Changed lines of the file:
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@@
     (pin "1")
+  )
+  (symbol (lib_id "ao_symbols:Graphic") (at 203.2 158.75 0) (unit 1)
+    (in_bom no) (on_board yes) (fields_autoplaced)
+    (property "Reference" "GRAF2" (id 0) (at 210.185 157.9153 0)
+      (effects (font (size 1.27 1.27)) (justify left))
+    )
+    (property "Value" "CC0 logo" (id 1) (at 210.185 160.4522 0)
+      (effects (font (size 1.27 1.27)) (justify left))
+    )
+    (property "Footprint" "ao_tht:CC0_logo" (id 2) (at 203.2 158.75 0)
+      (effects (font (size 1.27 1.27)) hide)
+    )
+    (property "Datasheet" "" (id 3) (at 203.2 158.75 0)
+      (effects (font (size 1.27 1.27)) hide)
+    )
+    (property "Config" "DNF" (id 4) (at 203.2 158.75 0)
+      (effects (font (size 1.27 1.27)) hide)
+    )
   )
   (symbol (lib_id "power:-12V") (at 88.9 187.96 180) (unit 1)
@@
     )
     (pin "1")
+  )
+  (symbol (lib_id "ao_symbols:Graphic") (at 203.2 165.1 0) (unit 1)
+    (in_bom no) (on_board yes) (fields_autoplaced)
+    (property "Reference" "GRAF3" (id 0) (at 210.185 164.2653 0)
+      (effects (font (size 1.27 1.27)) (justify left))
+    )
+    (property "Value" "AO logo" (id 1) (at 210.185 166.8022 0)
+      (effects (font (size 1.27 1.27)) (justify left))
+    )
+    (property "Footprint" "ao_tht:analogoutput" (id 2) (at 203.2 165.1 0)
+      (effects (font (size 1.27 1.27)) hide)
+    )
+    (property "Datasheet" "" (id 3) (at 203.2 165.1 0)
+      (effects (font (size 1.27 1.27)) hide)
+    )
+    (property "Config" "DNF" (id 4) (at 203.2 165.1 0)
+      (effects (font (size 1.27 1.27)) hide)
+    )
   )
   (symbol (lib_id "ao_symbols:2_pin_Molex_header") (at 62.23 91.44 180) (unit 1)
@@
       (reference "GRAF1") (unit 1) (value "Graphic") (footprint "mikrokosmos-ii:mikrokosmos-ii_panel_holes")
     )
+    (path "/022e93a0-8d56-459f-8a7d-1f4825b94da6"
+      (reference "GRAF2") (unit 1) (value "CC0 logo") (footprint "ao_tht:CC0_logo")
+    )
+    (path "/36619ae7-4265-4004-b610-d69b7bc9ab5d"
+      (reference "GRAF3") (unit 1) (value "AO logo") (footprint "ao_tht:analogoutput")
+    )
     (path "/2548420e-b440-45f5-9367-4aa430075ba1"

Commit message: panel, PCB updates
Parts:
- added H2: MountingHole, ao_tht:MountingHole_3.2mm_M3, symbol ao_symbols:MountingHole
Changed lines of the file:
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@@
+    )
+  )
+  (symbol (lib_id "ao_symbols:MountingHole") (at 53.34 132.08 0) (unit 1)
+    (in_bom no) (on_board yes) (fields_autoplaced)
+    (property "Reference" "H2" (id 0) (at 55.88 131.2453 0)
+      (effects (font (size 1.27 1.27)) (justify left))
+    )
+    (property "Value" "MountingHole" (id 1) (at 55.88 133.7822 0)
+      (effects (font (size 1.27 1.27)) (justify left))
+    )
+    (property "Footprint" "ao_tht:MountingHole_3.2mm_M3" (id 2) (at 53.34 132.08 0)
+      (effects (font (size 1.27 1.27)) hide)
+    )
+    (property "Datasheet" "" (id 3) (at 53.34 132.08 0)
+      (effects (font (size 1.27 1.27)) hide)
+    )
+    (property "Config" "DNF" (id 4) (at 53.34 132.08 0)
+      (effects (font (size 1.27 1.27)) hide)
     )
   )
@@
       (reference "H1") (unit 1) (value "MountingHole") (footprint "ao_tht:MountingHole_3.2mm_M3")
     )
+    (path "/2e4bef08-441e-4695-9f8d-6be7af5dd700"
+      (reference "H2") (unit 1) (value "MountingHole") (footprint "ao_tht:MountingHole_3.2mm_M3")
+    )
     (path "/c7ace7a6-8630-4d4f-a859-c36885f87241"

Commit message: Pre fab tweaks, Gerbers, cap descriptions
Parts:
- renumbered C2 to C1, C3 to C2, C1 to C3, C5 to C4, C6 to C5, C4 to C6, C10 to C8, C11 to C9, J6 to J3, J7 to J4, J4 to J5, J3 to J6, J5 to J7, R8 to R1, R1 to R2, R2 to R3, R3 to R4, R4 to R5, R5 to R6, R6 to R7, R7 to R8
